File: two_axis_balancing_carrier/two_axis_balancing_carrier.kicad_sch (KiCad schematic)
At the start: 27 parts, among them J1 Conn_01x03, J2 Conn_01x04, J5 Conn_02x05, U1 NUCLEO-G474RE, U2 MIC5219-3.3YM5, U3 ICM-42688-P, U4 SN65HVD230

Commit message: Connectors need changing
Parts:
- J1: footprint Connector_JST:JST_XH_B3B-XH-A_1x03_P2.50mm_Vertical -> Connector_JST:JST_GH_BM04B-GHS-TBT_1x04-1MP_P1.25mm_Vertical
Connections:
- net CANH: now also J1.3 (Pin_3); no longer J1.1 (Pin_1)
- net GND: now also J1.1 (Pin_1); no longer J1.3 (Pin_3)
Changed lines of the file:
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@@
 	(wire
 		(pts
+			(xy 264.16 35.56) (xy 254 35.56)
+		)
+		(stroke
+			(width 0)
+			(type default)
+		)
+	)
+	(wire
+		(pts
 			(xy 160.02 30.48) (xy 160.02 35.56)
 		)
@@
 	)
 	(label "CANH"
-		(at 254 35.56 0)
+		(at 254 40.64 0)
 		(effects
 			(font
@@
 	(symbol
 		(lib_id "power:GND")
-		(at 254 40.64 0)
+		(at 264.16 35.56 0)
 		(mirror y)
 		(unit 1)
@@
 		(fields_autoplaced yes)
 		(property "Reference" "#PWR013"
-			(at 254 46.99 0)
+			(at 264.16 41.91 0)
 			(hide yes)
 			(show_name no)
@@
 		)
 		(property "Value" "GND"
-			(at 254 45.72 0)
+			(at 266.7 36.8299 0)
 			(show_name no)
 			(do_not_autoplace no)
@@
 					(size 1.27 1.27)
 				)
+				(justify right)
 			)
 		)
 		(property "Footprint" ""
-			(at 254 40.64 0)
+			(at 264.16 35.56 0)
 			(hide yes)
 			(show_name no)
@@
 		)
 		(property "Datasheet" ""
-			(at 254 40.64 0)
+			(at 264.16 35.56 0)
 			(hide yes)
 			(show_name no)
@@
 		)
 		(property "Description" "Power symbol creates a global label with name \"GND\" , ground"
-			(at 254 40.64 0)
+			(at 264.16 35.56 0)
 			(hide yes)
 			(show_name no)
@@
 			)
 		)
-		(property "Footprint" "Connector_JST:JST_XH_B3B-XH-A_1x03_P2.50mm_Vertical"
+		(property "Footprint" "Connector_JST:JST_GH_BM04B-GHS-TBT_1x04-1MP_P1.25mm_Vertical"
 			(at 248.92 38.1 0)
 			(hide yes)

Commit message: Finished carrier prototype
Connections:
- net ENC_B: now also J2.4 (Pin_4); no longer J2.2 (Pin_2)
- net GND: now also J2.2 (Pin_2); no longer J2.4 (Pin_4)
Changed lines of the file:
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@@
+	(wire
+		(pts
+			(xy 254 69.85) (xy 265.43 69.85)
+		)
+		(stroke
+			(width 0)
+			(type default)
+		)
+	)
 	(wire
 		(pts
@@
 	)
 	(label "ENC_B"
-		(at 254 69.85 0)
+		(at 254 74.93 0)
 		(effects
 			(font
@@
 	(symbol
 		(lib_id "power:GND")
-		(at 254 74.93 0)
+		(at 265.43 69.85 0)
 		(unit 1)
 		(body_style 1)
@@
 		(fields_autoplaced yes)
 		(property "Reference" "#PWR016"
-			(at 254 81.28 0)
+			(at 265.43 76.2 0)
 			(hide yes)
 			(show_name no)
@@
 		)
 		(property "Value" "GND"
-			(at 254 80.01 0)
+			(at 265.43 74.93 0)
 			(show_name no)
 			(do_not_autoplace no)
@@
 		)
 		(property "Footprint" ""
-			(at 254 74.93 0)
+			(at 265.43 69.85 0)
 			(hide yes)
 			(show_name no)
@@
 		)
 		(property "Datasheet" ""
-			(at 254 74.93 0)
+			(at 265.43 69.85 0)
 			(hide yes)
 			(show_name no)
@@
 		)
 		(property "Description" "Power symbol creates a global label with name \"GND\" , ground"
-			(at 254 74.93 0)
-			(hide yes)
-			(show_name no)
+			(at 265.43 69.85 0)
+			(hide yes)
+			(show_name no)
