File: two_axis_balancing_carrier/two_axis_balancing_carrier.kicad_pcb (KiCad board)
At the start: 4 copper layers, 101.6 x 90.9 mm, 31 parts, among them J1 Conn_01x03, J2 Conn_01x04, J5 Conn_02x05, U1 NUCLEO-G474RE, U2 MIC5219-3.3YM5, U3 ICM-42688-P, U4 SN65HVD230

Commit message: Connectors need changing
Parts:
- J1: footprint Connector_PinSocket_2.54mm:PinSocket_1x03_P2.54mm_Vertical -> Connector_JST:JST_GH_BM04B-GHS-TBT_1x04-1MP_P1.25mm_Vertical
- J2: footprint Connector_PinSocket_2.54mm:PinSocket_1x04_P2.54mm_Vertical -> Connector_JST:JST_XH_B4B-XH-A_1x04_P2.50mm_Vertical
- moved J1 4.26 mm to (177.5, 64.1)
- moved R1 2.95 mm to (177.4, 69.7)
- moved C3 2.95 mm to (178.7, 78.8)
- moved U4 2.95 mm to (177.3, 74.2)
Connections:
- J1 pad 1: /CANH -> GND
- J1 pad 3: GND -> /CANH
Routing:
- net +3.3V: track 73.1 -> 44.9 mm
- net /RX: track 43.1 -> 34.1 mm
- net /CANH: track 9.37 -> 1.92 mm
- net /TX: track 35.7 -> 30.3 mm
- net /CANL: track 6.76 -> 1.77 mm
- net GND: vias 2 -> 92

Commit message: Finished carrier prototype
Parts:
- moved REF** 2.30 mm to (86.8, 143.5)
- moved J2 1.72 mm to (129.6, 143.4), turned to 180 degrees
- moved J1 0.18 mm to (177.3, 64.2), turned to 180 degrees
- renumbered TP2 to 3.3V, TP1 to 5V, TP7 to CS, TP12 to ENC_A, TP13 to ENC_B, TP3 to GND, TP9 to INT2, TP11 to RX, TP5 to SCLK, TP4 to SDI, TP6 to SDO, TP8 to TPINT1, TP10 to TX
Connections:
- J2 pad 2: /ENC_B -> GND
- J2 pad 4: GND -> /ENC_B
Routing:
- net +3.3V: track 44.9 -> 69.8 mm
- net /ENC_A: track 81.7 -> 98.0 mm
- net /CANL: track 1.77 -> 9.34 mm
- net /CANH: track 1.92 -> 9.45 mm
- net /RX: track 34.1 -> 39.4 mm
- net /ENC_B: track 57.1 -> 58.5 mm
- net /TX: track 30.3 -> 31.6 mm
- net +5V: track 176.5 -> 177.6 mm
- net GND: track 8.51 -> 8.71 mm, vias 92 -> 155
Other:
- board size 101.6 x 90.9 mm -> 101.6 x 92.9 mm

Commit message: Small fix
Parts:
- renumbered TPINT1 to INT1
Changed lines of the file:
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@@
 		(descr "SMD rectangular pad as test Point, square 2.0mm side length")
 		(tags "test point SMD pad rectangle square")
-		(property "Reference" "TPINT1"
+		(property "Reference" "INT1"
 			(at 0 -1.998 0)
 			(layer "F.SilkS")

Commit message: More small fixes
Routing:
- net +5V: track 177.6 -> 157.3 mm
- net GND: vias 155 -> 169
