File: hardware/two_axis_balancing_power/two_axis_balancing_power.kicad_sch (KiCad schematic)
At the start: 35 parts, among them J1 Conn_01x02, J2 Conn_02x05, J3 Conn_01x02, Q1 AO3401A, U1 RPL-1.0-R, U2 LM393, U3 TB6612FNG

Commit message: Fixed issue with battery monitoring functionality
Parts:
- added R11: 10kR, Resistor_SMD:R_0603_1608Metric, symbol Device:R_US
- added R12: 15kR, Resistor_SMD:R_0603_1608Metric, symbol Device:R_US
- added R9: 220kR, Resistor_SMD:R_0603_1608Metric, symbol Device:R_US
- R10: renamed from R9; value 220R -> 470R
- renumbered R10 to R13, R3 to R2, R4 to R3, R6 to R4, R7 to R5, R8 to R6, R2 to R7, R5 to R8, TP2 to TP5V1, TP5 to TPAIN1, TP6 to TPAIN2, TP8 to TPBLEV1, TP3 to TPGND1, TP9 to TPPG1, TP4 to TPPWMA1, TP7 to TPSTBY1, TP1 to TPVBAT1
Connections:
- net +5V: now also D2.2 (A), R3.1, R11.1; no longer R3.2
- net BAT_LEV: now also R8.2, TPBLEV1.1, U2.2 (-), U2.5 (+); no longer R8.1, U2.3 (+)
- net BAT_LOW: now also R11.2, R12.1, R9.1; no longer R10.2
- net GND: now also R8.1, R12.2; no longer D2.1 (K), R8.2
- net at R10.1: now also D2.1 (K); no longer D2.2 (A)
- net at U2.6 (-): now also R3.2, R4.1, U2.3 (+), R9.2
- net at U2.7: now also R10.2
- removed net BAT_REF: R3.1, R4.1, TPBLEV1.1, U2.2 (-)
Other:
- moved on the sheet: C5, C6, D2, J2, J3, R10, R3, R4, R7, R8, U2A, U2B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
