File: hardware/two_axis_balancing_carrier_mcu_version/two_axis_balancing_carrier_mcu_version/two_axis_balancing_carrier_mcu_version.kicad_sch (KiCad schematic)
At the start: 55 parts, among them J1 Conn_02x05, J2 Conn_ST_STDC14, J3 Conn_01x04, J4 Conn_01x04, J5 Conn_02x08_Odd_Even, U1 MIC5219-3.3YM5, U2 ICM-42688-P, U3 SN65HVD230, U4 STM32G474RETx, Y1 8MHz

Commit message: Started rev 2 of carrier board, mainly swapping the dev board for a bare mcu
Parts:
- C10, C11, C12, C13, C15, C19, C20, C21, C5, C6, C7, C8, FB1, FB2: footprint (none) -> Capacitor_SMD:C_0603_1608Metric
- C16, C3, C4: footprint (none) -> Capacitor_SMD:C_0805_2012Metric
- D1, D2: footprint (none) -> LED_SMD:LED_0603_1608Metric
- J2: footprint (none) -> Connector_PinHeader_1.27mm:PinHeader_2x07_P1.27mm_Vertical
- Y1: footprint (none) -> Crystal:Crystal_SMD_7050-4Pin_7.0x5.0mm
Connections:
- net +3.3V: now also J1.6 (Pin_6)
- net GND: no longer J1.6 (Pin_6)
Changed lines of the file:
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@@
 		)
 	)
-	(label "GND"
+	(label "+3.3V"
 		(at 59.69 45.72 0)
 		(effects
@@
 			)
 		)
-		(property "Footprint" ""
+		(property "Footprint" "Capacitor_SMD:C_0603_1608Metric"
 			(at 144.78 168.91 0)
 			(hide yes)
@@
 			)
 		)
-		(property "Footprint" ""
+		(property "Footprint" "Capacitor_SMD:C_0603_1608Metric"
 			(at 137.16 150.622 90)
 			(hide yes)
@@
 			)
 		)
-		(property "Footprint" ""
+		(property "Footprint" "LED_SMD:LED_0603_1608Metric"
 			(at 229.87 219.71 0)
 			(hide yes)
@@
 			)
 		)
-		(property "Footprint" ""
+		(property "Footprint" "Capacitor_SMD:C_0603_1608Metric"
 			(at 130.81 138.43 0)
 			(hide yes)
@@
 			)
 		)
-		(property "Footprint" ""
+		(property "Footprint" "Capacitor_SMD:C_0603_1608Metric"
 			(at 176.53 151.13 0)
 			(hide yes)
@@
 			)
 		)
-		(property "Footprint" ""
+		(property "Footprint" "Capacitor_SMD:C_0805_2012Metric"
 			(at 142.24 154.94 0)
 			(hide yes)
@@
 			)
 		)
-		(property "Footprint" ""
+		(property "Footprint" "Capacitor_SMD:C_0603_1608Metric"
 			(at 259.08 246.38 0)
 			(hide yes)
@@
 			)
 		)
-		(property "Footprint" ""
+		(property "Footprint" "Capacitor_SMD:C_0603_1608Metric"
 			(at 144.78 176.53 0)
 			(hide yes)
@@
 			)
 		)
-		(property "Footprint" ""
+		(property "Footprint" "Capacitor_SMD:C_0603_1608Metric"
 			(at 199.898 146.05 90)
 			(hide yes)
@@
 			)
 		)
-		(property "Footprint" ""
+		(property "Footprint" "Capacitor_SMD:C_0603_1608Metric"
 			(at 245.11 177.8 0)
 			(hide yes)
@@
 			)
 		)
-		(property "Footprint" ""
+		(property "Footprint" "Crystal:Crystal_SMD_7050-4Pin_7.0x5.0mm"
 			(at 158.75 172.72 0)
 			(hide yes)
@@
 			)
 		)
-		(property "Footprint" ""
+		(property "Footprint" "Capacitor_SMD:C_0805_2012Metric"
 			(at 119.38 138.43 0)
 			(hide yes)
@@
 			)
 		)
-		(property "Footprint" ""
+		(property "Footprint" "Capacitor_SMD:C_0603_1608Metric"
 			(at 259.08 231.14 0)
 			(hide yes)
@@
 			)
 		)
-		(property "Footprint" ""
+		(property "Footprint" "Capacitor_SMD:C_0603_1608Metric"
 			(at 153.67 154.94 0)
 			(hide yes)
@@
 			)
 		)
-		(property "Footprint" ""
+		(property "Footprint" "Capacitor_SMD:C_0805_2012Metric"
 			(at 228.6 153.67 0)
 			(hide yes)
@@
 			)
 		)
-		(property "Footprint" ""
+		(property "Footprint" "Connector_PinHeader_1.27mm:PinHeader_2x07_P1.27mm_Vertical"
 			(at 264.16 190.5 0)
 			(hide yes)
@@
 			)
 		)
-		(property "Footprint" ""
+		(property "Footprint" "Capacitor_SMD:C_0603_1608Metric"
 			(at 153.67 138.43 0)
 			(hide yes)
@@
 			)
 		)
-		(property "Footprint" ""
+		(property "Footprint" "Capacitor_SMD:C_0603_1608Metric"
 			(at 214.63 153.67 0)
 			(hide yes)
@@
 			)
 		)
-		(property "Footprint" ""
+		(property "Footprint" "Capacitor_SMD:C_0603_1608Metric"
 			(at 166.37 138.43 0)
 			(hide yes)
@@
 			)
 		)
-		(property "Footprint" ""
+		(property "Footprint" "LED_SMD:LED_0603_1608Metric"
 			(at 229.87 215.9 0)
 			(hide yes)
@@
 			)
 		)
-		(property "Footprint" ""
+		(property "Footprint" "Capacitor_SMD:C_0603_1608Metric"
 			(at 142.24 138.43 0)
 			(hide yes)

Commit message: Nearly finished layout and routing
Parts:
- added C5: 1uF, Capacitor_SMD:C_0603_1608Metric, symbol Device:C
- Y1: footprint Crystal:Crystal_SMD_7050-4Pin_7.0x5.0mm -> Crystal:Crystal_SMD_3225-4Pin_3.2x2.5mm
- renumbered C14 to C1, C13 to C12, C12 to C13, C15 to C14, C16 to C15, C4 to C16, C8 to C17, C6 to C18, C7 to C19, C9 to C2, C21 to C20, C19 to C21, C20 to C22, C17 to C3, C18 to C4, C2 to C6, C1 to C7, C3 to C8, C5 to C9, FB2 to FB1, FB1 to FB2, J3 to J1, J1 to J2, J4 to J3, J2 to J4, R2 to R1, R1 to R2, TP12 to TP10, TP6 to TP11, TP13 to TP12, TP7 to TP13, TP8 to TP2, TP2 to TP3, TP9 to TP4, TP3 to TP5, TP10 to TP6, TP4 to TP7, TP11 to TP8, TP5 to TP9, U3 to U1, U1 to U3
Connections:
- net +5V: now also C5.1
- net GND: now also C5.2
- net LED_HB: now reaches U4.38 (PC6)
- net LED_HB: now also R3.1
- net at U4.57 (PB4): no longer R3.1
- net LED_FAULT: now reaches R4.1
- net LED_FAULT: now also U4.42 (PA8); no longer U4.58 (PB5)
- net PA8 renamed PB5
- net PB5: now also U4.58 (PB5); no longer U4.42 (PA8)
Other:
- moved on the sheet: C20, D1, D2, J4, R3, R4

Commit message: nearly finished layout and routing
Parts:
- added C23: 100nF, Capacitor_SMD:C_0603_1608Metric, symbol Device:C_Small
- added TP14: TestPoint, TestPoint:TestPoint_Keystone_5015_Micro_Mini, symbol Connector:TestPoint
- TP1, TP10, TP11, TP12, TP13, TP2, TP3, TP4, TP6, TP7, TP8, TP9: footprint TestPoint:TestPoint_Pad_2.0x2.0mm -> TestPoint:TestPoint_Pad_D1.0mm
- TP5: footprint TestPoint:TestPoint_Pad_2.0x2.0mm -> TestPoint:TestPoint_Keystone_5015_Micro_Mini
Connections:
- net BAT_LEV: now also C23.1
- net GND: now also C23.2, TP14.1
- net PA10: now also J5.12 (Pin_12); no longer J5.8 (Pin_8)
- net PA9: now also J5.11 (Pin_11); no longer J5.7 (Pin_7)
- net PB10: now also J5.7 (Pin_7); no longer J5.13 (Pin_13)
- net PB11: now also J5.8 (Pin_8); no longer J5.14 (Pin_14)
- net PB5: now also J5.16 (Pin_16); no longer J5.12 (Pin_12)
- net PC10: now also J5.13 (Pin_13); no longer J5.9 (Pin_9)
- net PC11: now also J5.14 (Pin_14); no longer J5.10 (Pin_10)
- net PC12: now also J5.15 (Pin_15); no longer J5.11 (Pin_11)
- net PC4: now also J5.5 (Pin_5); no longer J5.15 (Pin_15)
- net PC5: now also J5.6 (Pin_6); no longer J5.16 (Pin_16)
- net PC8: now also J5.9 (Pin_9); no longer J5.5 (Pin_5)
- net PC9: now also J5.10 (Pin_10); no longer J5.6 (Pin_6)
Other:
- moved on the sheet: C20, C21, C22, D1, D2, J4, R3, R4, R6, R7

Commit message: breakout header routing reworked
Connections:
- net PA10: now also J5.10 (Pin_10); no longer J5.12 (Pin_12)
- net PA9: now also J5.9 (Pin_9); no longer J5.11 (Pin_11)
- net PB10: now also J5.8 (Pin_8); no longer J5.7 (Pin_7)
- net PB11: now also J5.7 (Pin_7); no longer J5.8 (Pin_8)
- net PC8: now also J5.11 (Pin_11); no longer J5.9 (Pin_9)
- net PC9: now also J5.12 (Pin_12); no longer J5.10 (Pin_10)
Changed lines of the file:
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@@
 	)
 	(label "PC8"
-		(at 350.52 207.01 180)
+		(at 350.52 209.55 180)
 		(effects
 			(font
@@
 	)
 	(label "PB10"
-		(at 350.52 204.47 180)
-		(effects
-			(font
-				(size 1.27 1.27)
-			)
-			(justify right bottom)
+		(at 363.22 204.47 0)
+		(effects
+			(font
+				(size 1.27 1.27)
+			)
+			(justify left bottom)
 		)
 	)
@@
 	)
 	(label "PA9"
-		(at 350.52 209.55 180)
+		(at 350.52 207.01 180)
 		(effects
 			(font
@@
 	)
 	(label "PC9"
-		(at 363.22 207.01 0)
+		(at 363.22 209.55 0)
 		(effects
 			(font
@@
 	)
 	(label "PB11"
-		(at 363.22 204.47 0)
-		(effects
-			(font
-				(size 1.27 1.27)
-			)
-			(justify left bottom)
+		(at 350.52 204.47 180)
+		(effects
+			(font
+				(size 1.27 1.27)
+			)
+			(justify right bottom)
 		)
 	)
@@
 	)
 	(label "PA10"
-		(at 363.22 209.55 0)
-		(effects
-			(font
+		(at 363.22 207.01 0)
+		(effects
+			(font
